Commit message: nodelet dynamic_reconfigure

File: ros_gazebo/xacro/car.urdf (robot description, URDF)
Before this commit: robot car_xacro, 5 links, 4 joints
Links:
- added link laser; visual cylinder length=0.05 radius=0.03
- added link support; visual cylinder length=0.15 radius=0.01
- link camera: geometry visual box size=0.02 0.05 0.05
Joints:
- added joint laser: type fixed, parent base, child laser, origin xyz=0 0 0.20249999999999999 rpy=0 0 0
- added joint support: type fixed, parent base, child support, origin xyz=0 0 0.1025 rpy=0 0 0
- joint camera2base: origin (none) -> xyz=0.08 0 0.052500000000000005 rpy=0 0 0

File: rospy_urdf_learn/urdf/xacro/car.xacro (robot description, xacro)
@@ -5,4 +5,7 @@
     <xacro:include filename = "$(find rospy_urdf_learn)/urdf/xacro/car_base.xacro" />
     <xacro:include filename = "$(find rospy_urdf_learn)/urdf/xacro/car_joint.xacro" />
+    <!--包含摄像头和激光雷达xacro文件-->
+    <xacro:include filename = "$(find rospy_urdf_learn)/urdf/xacro/camera.xacro" />
+    <xacro:include filename = "$(find rospy_urdf_learn)/urdf/xacro/laser.xacro" />
     <!--参数-->
     <xacro:car_base name = "base"/>
