Commit message: roscontrol

File: rospy_urdf_learn/urdf/xacro/car.xacro (robot description, xacro)
@@ -1,4 +1,7 @@
 <?xml version = "1.0" ?>
 <robot name = "car_xacro" xmlns:xacro = "http://wiki.ros.org/xacro" >
+    <!--必要的参数-->
+    <xacro:property name = "wheel_radius" value = "0.0325" />
+    <xacro:property name = "base_link_radius" value = "0.1" />
     <!--导入操作-->
     <xacro:include filename = "$(find rospy_urdf_learn)/urdf/xacro/car_wheel.xacro" />
@@ -8,6 +11,9 @@
     <xacro:include filename = "$(find rospy_urdf_learn)/urdf/xacro/camera.xacro" />
     <xacro:include filename = "$(find rospy_urdf_learn)/urdf/xacro/laser.xacro" />
-    <!--参数-->
+    <!--运动控制包含-->
+    <xacro:include filename = "gazebo/move.xacro" />
+    <!--车的底盘-->
     <xacro:car_base name = "base"/>
+    <!--车的轮子实现-->
     <xacro:car_wheel name = "left_wheel" radius = "0.0325" length = "0.015" />
     <xacro:car_continuous_joint name = "left2base"
@@ -24,3 +30,8 @@
     rx = "0" ry = "0" rz = "1"
     />
+    <!--传动装置的实现-->
+    <xacro:joint_trans joint_name = "left2base" />
+    <xacro:joint_trans joint_name = "right2base" />
+    <!--导入雷达相关信息-->
+    <xacro:include filename = "$(find rospy_urdf_learn)/urdf/xacro/leida.xacro" />
 </robot>
